File: connector_pins.kicad_sch (KiCad schematic)
At the start: 4 parts, among them J1 Conn_01x04_Pin, J2 Conn_01x04_Pin, J3 Conn_01x09_Pin, J4 Conn_02x03_Odd_Even

Commit message: drew proper shape of board & routed circuits partially
Changed lines of the file:
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@@
 		)
 		(property "Description" "Serial UART"
-			(at 104.14 48.26 0)
+			(at 107.95 48.26 0)
 			(effects
 				(font
